File: drv_lfpak33.sch (KiCad schematic (older format))
At the start: 43 parts, among them J1 Conn_01x04_Male, J2 Conn_01x02_Male, J3 Conn_01x09_Male, J4 Conn_01x02_Male, Q1 PSMN1R8-30MLH, Q2 PSMN1R8-30MLH, Q3 PSMN1R8-30MLH, Q4 PSMN1R8-30MLH, Q5 PSMN1R8-30MLH, Q6 PSMN1R8-30MLH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

Commit message: update schematic: correct pull resistor values
Parts:
- R12, R2, R7: value 2k7 (8k66) -> 3k9 (8k66)
Other:
- note added: "R1,R2 and equivalent resistors for phases B and C:\n\nFor two plain open drain outputs pulling low,\npopulate both (suggestion: 3k9 to 5V, 2k7 to _H input)\n\nThe values in parantheses are for\n- open drain pulling low\n- open drain with internal series resistor pulling low\ntied together on AL (PSoC6)"
- note removed: "R1,R2 and equivalent resistors for phases B and C:\n\nFor two plain open drain outputs pulling low,\npopulate both with equal values (suggestion: 2k7)\n\nThe values in parantheses are for\n- open drain pulling low\n- open drain with internal series resistor pulling low\ntied together on AL (tested with PSoC6)"
Changed lines of the file:
@@
 P 3500 1350
 F 0 "R2" H 3559 1396 50  0000 L CNN
-F 1 "2k7 (8k66)" H 3559 1305 50  0000 L CNN
+F 1 "3k9 (8k66)" H 3559 1305 50  0000 L CNN
 F 2 "Resistor_SMD:R_0603_1608Metric" H 3500 1350 50  0001 C CNN
 F 3 "~" H 3500 1350 50  0001 C CNN
@@
 P 3500 3200
 F 0 "R7" H 3559 3246 50  0000 L CNN
-F 1 "2k7 (8k66)" H 3559 3155 50  0000 L CNN
+F 1 "3k9 (8k66)" H 3559 3155 50  0000 L CNN
 F 2 "Resistor_SMD:R_0603_1608Metric" H 3500 3200 50  0001 C CNN
 F 3 "~" H 3500 3200 50  0001 C CNN
@@
 P 3500 5050
 F 0 "R12" H 3559 5096 50  0000 L CNN
-F 1 "2k7 (8k66)" H 3559 5005 50  0000 L CNN
+F 1 "3k9 (8k66)" H 3559 5005 50  0000 L CNN
 F 2 "Resistor_SMD:R_0603_1608Metric" H 3500 5050 50  0001 C CNN
 F 3 "~" H 3500 5050 50  0001 C CNN
@@
 see note at bottom
 Text Notes 4700 7300 0    50   ~ 0
-R1,R2 and equivalent resistors for phases B and C:\n\nFor two plain open drain outputs pulling low,\npopulate both with equal values (suggestion: 2k7)\n\nThe values in parantheses are for\n- open drain pulling low\n- open drain with internal series resistor pulling low\ntied together on AL (tested with PSoC6)
+R1,R2 and equivalent resistors for phases B and C:\n\nFor two plain open drain outputs pulling low,\npopulate both (suggestion: 3k9 to 5V, 2k7 to _H input)\n\nThe values in parantheses are for\n- open drain pulling low\n- open drain with internal series resistor pulling low\ntied together on AL (PSoC6)
 Text Notes 8200 6250 0    50   ~ 0
 Close J2 with jumper for "classic" gnd referenced voltage dividers

Commit message: add mounting holes
Parts:
- added H1, H2: MountingHole, MountingHole:MountingHole_3.2mm_M3, symbol Mechanical:MountingHole
Changed lines of the file:
@@
 Text Notes 8250 2100 0    50   ~ 0
 Voltage dividers:\n10k / 2k2 for up to 3S\n10k / 1k for up to 6S
+$Comp
+L Mechanical:MountingHole H1
+U 1 1 60DBA222
+P 1450 5550
+F 0 "H1" H 1550 5596 50  0000 L CNN
+F 1 "MountingHole" H 1550 5505 50  0000 L CNN
+F 2 "MountingHole:MountingHole_3.2mm_M3" H 1450 5550 50  0001 C CNN
+F 3 "~" H 1450 5550 50  0001 C CNN
+	1    1450 5550
+	1    0    0    -1
+$EndComp
+$Comp
+L Mechanical:MountingHole H2
+U 1 1 60DBE191
+P 1450 5750
+F 0 "H2" H 1550 5796 50  0000 L CNN
+F 1 "MountingHole" H 1550 5705 50  0000 L CNN
+F 2 "MountingHole:MountingHole_3.2mm_M3" H 1450 5750 50  0001 C CNN
+F 3 "~" H 1450 5750 50  0001 C CNN
+	1    1450 5750
+	1    0    0    -1
+$EndComp
 $EndSCHEMATC
